File: KiCad/isa_svga.sch (KiCad schematic (older format))
At the start: 62 parts, among them P1 VGA, U1 TVGA9000I, U2 27C256, U3 MT4C4256, U4 MT4C4256, U5 MT4C4256, U6 MT4C4256, X1 40MHz

Commit message: Add v1.1 files
Signed-off-by: Sergey Kiselev <skiselev@gmail.com>
Parts:
- removed X1: 40MHz, symbol CRYSTAL
- added X1: 40MHz, my_components:Crystal_HC-49U_Vert, symbol Crystal
- BUS1: footprint (none) -> my_components:Conn_Edge_ISA8
- C1, C10, C11, C12, C18, C19, C2, C20, C21, C22, C23, C24, C25, C26, C27, C3, C4, C5, C6, C7, C8, C9: footprint (none) -> my_components:Cap_Cer_508
- C13, C14, C15, C16: footprint (none) -> my_components:Cap_Tant_508
- C17: value 1nF -> 1uF; footprint (none) -> my_components:Cap_Cer_508
- FB1, FB2, FB3, FB4, FB5, FB6, L1, L2, L3: footprint (none) -> my_components:Res_1016
- JP1: footprint (none) -> my_components:Conn_Pin_Header_2x1_2.54mm_NoKey
- P1: footprint (none) -> my_components:Conn_Dsub_DE15F
- R1, R10, R11, R12, R13, R14, R15, R16, R2, R3, R4, R5, R6, R7, R8, R9: footprint (none) -> my_components:Res_762
- U1: footprint (none) -> my_components:IC_PQFP-160
- U2: footprint (none) -> my_components:IC_DIP28_600
- U3, U4, U5, U6: footprint (none) -> my_components:IC_DIP20_300
Connections:
- net labels removed: ALE
- wire segments 396 -> 395
- no-connect marks 49 -> 50
